Commit message: fix: urdf

File: src/nexus_4wd_mecanum_simulator/nexus_4wd_mecanum_description/urdf/nexus_4wd_mecanum.xacro (robot description, xacro)
@@ -43,5 +43,5 @@
     <child link="upper_left_wheel_shaft" />
   </joint>
-  <link name="upper_left_wheel_shaft">
+  <link name="upper_left_wheel_shaft" >
     <visual>
       <origin xyz="0 0 0" rpy="0 0 0" />
@@ -150,5 +150,5 @@
     </inertial>
   </link>
-  <joint name="upper_left_wheel_joint" type="continuous">
+  <joint name="upper_left_wheel_joint" type="fixed">
     <origin xyz="0 0.042 0" rpy="0 0 0" />
     <parent link="upper_left_wheel_shaft"/>
@@ -180,5 +180,5 @@
     </inertial>
   </link>
-  <joint name="lower_left_wheel_joint" type="continuous">
+  <joint name="lower_left_wheel_joint" type="fixed">
     <origin xyz="0 0.042 0" rpy="0 0 0" />
     <parent link="lower_left_wheel_shaft"/>
@@ -210,5 +210,5 @@
     </inertial>
   </link>
-  <joint name="upper_right_wheel_joint" type="continuous">
+  <joint name="upper_right_wheel_joint" type="fixed">
     <origin xyz="0 0.042 0" rpy="0 0 0" />
     <parent link="upper_right_wheel_shaft"/>
@@ -240,5 +240,5 @@
     </inertial>
   </link>
-  <joint name="lower_right_wheel_joint" type="continuous">
+  <joint name="lower_right_wheel_joint" type="fixed">
     <origin xyz="0 0.042 0" rpy="0 0 0" />
     <parent link="lower_right_wheel_shaft"/>
@@ -322,4 +322,18 @@
       <geometry>
         <mesh filename="package://nexus_4wd_mecanum_description/meshes/urm04.STL" scale="0.001 0.001 0.001"/>
+      </geometry>
+      <material name="black" />
+    </visual>
+  </link>
+  <joint name="stereo_camera_joint" type="fixed">
+    <origin xyz="0.205 0 0.010" rpy="0 0 0" />
+    <parent link="base_link"/>
+    <child link="stereo_camera" />
+  </joint>
+  <link name="stereo_camera">
+    <visual>
+      <origin xyz="0 0 0" rpy="0 0 0" />
+      <geometry>
+        <box size="0.02 0.08 0.01" />
       </geometry>
       <material name="black" />
@@ -338,3 +352,6 @@
   <!-- rear sensor -->
   <xacro:urm04_sensor frame_name="rear_sensor" ros_topic="rear_sensor" update_rate="10" min_range="0.04" max_range="2.5" horizontal_field_of_view="1.04" vertical_field_of_view="0.04" ray_count="2" />
+  <!-- Include stereo camera -->
+  <xacro:include filename="$(find nexus_4wd_mecanum_description)/urdf/stereo_camera.xacro"/>
+  <xacro:stereo_camera frame_name="stereo_camera" ros_topic="stereo_camera" update_rate="30" width="800" height="600"/>
 </robot>
